Commit message: EXPERIMENTAL: add world joint to robot
This is required for planning with whole-motion planning with moveit.

File: tiago_description/robots/tiago_steel.urdf.xacro (robot description, xacro)
@@ -36,3 +36,8 @@
     <origin xyz="0.01 0 0" rpy="${90*deg_to_rad} ${90*deg_to_rad} ${-90*deg_to_rad}"/>
   </xacro:pal_gripper>
+  <link name="world" />
+  <joint type="planar" name="world_joint">
+    <parent link="world" />
+    <child link="base_footprint" />
+  </joint>
 </robot>
